Commit message: Reorganização geral dos launch files

File: remy_description/urdf/urdf2.xacro (robot description, xacro)
@@ -1,7 +1,7 @@
 <?xml version="1.0" ?>
 <robot name="urdf2" xmlns:xacro="http://www.ros.org/wiki/xacro">
-<xacro:include filename="$(find urdf2_description)/urdf/materials.xacro" />
-<xacro:include filename="$(find urdf2_description)/urdf/urdf2.trans" />
-<xacro:include filename="$(find urdf2_description)/urdf/urdf2.gazebo" />
+<xacro:include filename="$(find remy_description)/urdf/materials.xacro" />
+<xacro:include filename="$(find remy_description)/urdf/urdf2.trans" />
+<xacro:include filename="$(find remy_description)/urdf/urdf2.gazebo" />
 <link name="base_footprint"/>
 <!-- base_link agora é só um frame de referência (o que o diff_drive_controller
@@ -33,5 +33,5 @@
     <origin xyz="0 0 0" rpy="0 0 0"/>
     <geometry>
-      <mesh filename="file://$(find urdf2_description)/meshes/base_link.stl" scale="0.001 0.001 0.001"/>
+      <mesh filename="file://$(find remy_description)/meshes/base_link.stl" scale="0.001 0.001 0.001"/>
     </geometry>
     <material name="silver"/>
@@ -55,5 +55,5 @@
     <origin xyz="-0.0215 0.190948 -0.125363" rpy="0 0 0"/>
     <geometry>
-      <mesh filename="file://$(find urdf2_description)/meshes/limb2_v1_1.stl" scale="0.001 0.001 0.001"/>
+      <mesh filename="file://$(find remy_description)/meshes/limb2_v1_1.stl" scale="0.001 0.001 0.001"/>
     </geometry>
     <material name="silver"/>
@@ -77,5 +77,5 @@
     <origin xyz="-0.0325 -0.0265 -1.500001" rpy="0 0 0"/>
     <geometry>
-      <mesh filename="file://$(find urdf2_description)/meshes/limb3_v1_1.stl" scale="0.001 0.001 0.001"/>
+      <mesh filename="file://$(find remy_description)/meshes/limb3_v1_1.stl" scale="0.001 0.001 0.001"/>
     </geometry>
     <material name="silver"/>
@@ -99,5 +99,5 @@
     <origin xyz="-0.2235 -0.0 -0.074" rpy="0 0 0"/>
     <geometry>
-      <mesh filename="file://$(find urdf2_description)/meshes/limb1_v1_1.stl" scale="0.001 0.001 0.001"/>
+      <mesh filename="file://$(find remy_description)/meshes/limb1_v1_1.stl" scale="0.001 0.001 0.001"/>
     </geometry>
     <material name="silver"/>
@@ -120,5 +120,5 @@
     <origin xyz="0.2245 0.0 -0.074" rpy="0 0 0"/>
     <geometry>
-      <mesh filename="file://$(find urdf2_description)/meshes/limb1_v1__1__1.stl" scale="0.001 0.001 0.001"/>
+      <mesh filename="file://$(find remy_description)/meshes/limb1_v1__1__1.stl" scale="0.001 0.001 0.001"/>
     </geometry>
     <material name="silver"/>
@@ -142,5 +142,5 @@
     <origin xyz="0.09 0.12 -0.093" rpy="0 0 0"/>
     <geometry>
-      <mesh filename="file://$(find urdf2_description)/meshes/limb4_v1_1.stl" scale="0.001 0.001 0.001"/>
+      <mesh filename="file://$(find remy_description)/meshes/limb4_v1_1.stl" scale="0.001 0.001 0.001"/>
     </geometry>
     <material name="silver"/>
@@ -162,5 +162,5 @@
     <origin xyz="-0.09 -0.12 -0.093" rpy="0 0 0"/>
     <geometry>
-      <mesh filename="file://$(find urdf2_description)/meshes/limb4_v1__1__1.stl" scale="0.001 0.001 0.001"/>
+      <mesh filename="file://$(find remy_description)/meshes/limb4_v1__1__1.stl" scale="0.001 0.001 0.001"/>
     </geometry>
     <material name="silver"/>
@@ -182,5 +182,5 @@
     <origin xyz="0.09 -0.12 -0.093" rpy="0 0 0"/>
     <geometry>
-      <mesh filename="file://$(find urdf2_description)/meshes/limb4_v1__2__1.stl" scale="0.001 0.001 0.001"/>
+      <mesh filename="file://$(find remy_description)/meshes/limb4_v1__2__1.stl" scale="0.001 0.001 0.001"/>
     </geometry>
     <material name="silver"/>
@@ -202,5 +202,5 @@
     <origin xyz="-0.09 0.12 -0.093" rpy="0 0 0"/>
     <geometry>
-      <mesh filename="file://$(find urdf2_description)/meshes/limb4_v1__3__1.stl" scale="0.001 0.001 0.001"/>
+      <mesh filename="file://$(find remy_description)/meshes/limb4_v1__3__1.stl" scale="0.001 0.001 0.001"/>
     </geometry>
     <material name="silver"/>
@@ -223,5 +223,5 @@
     <origin xyz="0.068 0.145 -0.0331" rpy="0 0 0"/>
     <geometry>
-      <mesh filename="file://$(find urdf2_description)/meshes/limb5_v1_1.stl" scale="0.001 0.001 0.001"/>
+      <mesh filename="file://$(find remy_description)/meshes/limb5_v1_1.stl" scale="0.001 0.001 0.001"/>
     </geometry>
     <material name="silver"/>
@@ -243,5 +243,5 @@
     <origin xyz="-0.112 0.145 -0.0331" rpy="0 0 0"/>
     <geometry>
-      <mesh filename="file://$(find urdf2_description)/meshes/limb5_v1__1__1.stl" scale="0.001 0.001 0.001"/>
+      <mesh filename="file://$(find remy_description)/meshes/limb5_v1__1__1.stl" scale="0.001 0.001 0.001"/>
     </geometry>
     <material name="silver"/>
@@ -263,5 +263,5 @@
     <origin xyz="-0.112 -0.095 -0.0331" rpy="0 0 0"/>
     <geometry>
-      <mesh filename="file://$(find urdf2_description)/meshes/limb5_v1__2__1.stl" scale="0.001 0.001 0.001"/>
+      <mesh filename="file://$(find remy_description)/meshes/limb5_v1__2__1.stl" scale="0.001 0.001 0.001"/>
     </geometry>
     <material name="silver"/>
@@ -283,5 +283,5 @@
     <origin xyz="0.068 -0.095 -0.0331" rpy="0 0 0"/>
     <geometry>
-      <mesh filename="file://$(find urdf2_description)/meshes/limb5_v1__3__1.stl" scale="0.001 0.001 0.001"/>
+      <mesh filename="file://$(find remy_description)/meshes/limb5_v1__3__1.stl" scale="0.001 0.001 0.001"/>
     </geometry>
     <material name="silver"/>

File: remy_description/urdf/urdf2_quasebom.xacro (robot description, xacro)
@@ -1,7 +1,7 @@
 <?xml version="1.0" ?>
 <robot name="urdf2" xmlns:xacro="http://www.ros.org/wiki/xacro">
-<xacro:include filename="$(find urdf2_description)/urdf/materials.xacro" />
-<xacro:include filename="$(find urdf2_description)/urdf/urdf2.trans" />
-<xacro:include filename="$(find urdf2_description)/urdf/urdf2.gazebo" />
+<xacro:include filename="$(find remy_description)/urdf/materials.xacro" />
+<xacro:include filename="$(find remy_description)/urdf/urdf2.trans" />
+<xacro:include filename="$(find remy_description)/urdf/urdf2.gazebo" />
 <link name="base_footprint"/>
 <joint name="base_joint" type="fixed">
@@ -20,5 +20,5 @@
     <origin xyz="0 0 0" rpy="0 0 0"/>
     <geometry>
-      <mesh filename="file://$(find urdf2_description)/meshes/base_link.stl" scale="0.001 0.001 0.001"/>
+      <mesh filename="file://$(find remy_description)/meshes/base_link.stl" scale="0.001 0.001 0.001"/>
     </geometry>
     <material name="silver"/>
@@ -42,5 +42,5 @@
     <origin xyz="-0.0215 0.190948 -0.125363" rpy="0 0 0"/>
     <geometry>
-      <mesh filename="file://$(find urdf2_description)/meshes/limb2_v1_1.stl" scale="0.001 0.001 0.001"/>
+      <mesh filename="file://$(find remy_description)/meshes/limb2_v1_1.stl" scale="0.001 0.001 0.001"/>
     </geometry>
     <material name="silver"/>
@@ -64,5 +64,5 @@
     <origin xyz="-0.0325 -0.0265 -1.500001" rpy="0 0 0"/>
     <geometry>
-      <mesh filename="file://$(find urdf2_description)/meshes/limb3_v1_1.stl" scale="0.001 0.001 0.001"/>
+      <mesh filename="file://$(find remy_description)/meshes/limb3_v1_1.stl" scale="0.001 0.001 0.001"/>
     </geometry>
     <material name="silver"/>
@@ -86,5 +86,5 @@
     <origin xyz="-0.2235 -0.0 -0.074" rpy="0 0 0"/>
     <geometry>
-      <mesh filename="file://$(find urdf2_description)/meshes/limb1_v1_1.stl" scale="0.001 0.001 0.001"/>
+      <mesh filename="file://$(find remy_description)/meshes/limb1_v1_1.stl" scale="0.001 0.001 0.001"/>
     </geometry>
     <material name="silver"/>
@@ -107,5 +107,5 @@
     <origin xyz="0.2245 0.0 -0.074" rpy="0 0 0"/>
     <geometry>
-      <mesh filename="file://$(find urdf2_description)/meshes/limb1_v1__1__1.stl" scale="0.001 0.001 0.001"/>
+      <mesh filename="file://$(find remy_description)/meshes/limb1_v1__1__1.stl" scale="0.001 0.001 0.001"/>
     </geometry>
     <material name="silver"/>
@@ -130,5 +130,5 @@
     <origin xyz="0.09 0.12 -0.093" rpy="0 0 0"/>
     <geometry>
-      <mesh filename="file://$(find urdf2_description)/meshes/limb4_v1_1.stl" scale="0.001 0.001 0.001"/>
+      <mesh filename="file://$(find remy_description)/meshes/limb4_v1_1.stl" scale="0.001 0.001 0.001"/>
     </geometry>
     <material name="silver"/>
@@ -150,5 +150,5 @@
     <origin xyz="-0.09 -0.12 -0.093" rpy="0 0 0"/>
     <geometry>
-      <mesh filename="file://$(find urdf2_description)/meshes/limb4_v1__1__1.stl" scale="0.001 0.001 0.001"/>
+      <mesh filename="file://$(find remy_description)/meshes/limb4_v1__1__1.stl" scale="0.001 0.001 0.001"/>
     </geometry>
     <material name="silver"/>
@@ -170,5 +170,5 @@
     <origin xyz="0.09 -0.12 -0.093" rpy="0 0 0"/>
     <geometry>
-      <mesh filename="file://$(find urdf2_description)/meshes/limb4_v1__2__1.stl" scale="0.001 0.001 0.001"/>
+      <mesh filename="file://$(find remy_description)/meshes/limb4_v1__2__1.stl" scale="0.001 0.001 0.001"/>
     </geometry>
     <material name="silver"/>
@@ -190,5 +190,5 @@
     <origin xyz="-0.09 0.12 -0.093" rpy="0 0 0"/>
     <geometry>
-      <mesh filename="file://$(find urdf2_description)/meshes/limb4_v1__3__1.stl" scale="0.001 0.001 0.001"/>
+      <mesh filename="file://$(find remy_description)/meshes/limb4_v1__3__1.stl" scale="0.001 0.001 0.001"/>
     </geometry>
     <material name="silver"/>
@@ -212,5 +212,5 @@
     <origin xyz="0.068 0.145 -0.0331" rpy="0 0 0"/>
     <geometry>
-      <mesh filename="file://$(find urdf2_description)/meshes/limb5_v1_1.stl" scale="0.001 0.001 0.001"/>
+      <mesh filename="file://$(find remy_description)/meshes/limb5_v1_1.stl" scale="0.001 0.001 0.001"/>
     </geometry>
     <material name="silver"/>
@@ -232,5 +232,5 @@
     <origin xyz="-0.112 0.145 -0.0331" rpy="0 0 0"/>
     <geometry>
-      <mesh filename="file://$(find urdf2_description)/meshes/limb5_v1__1__1.stl" scale="0.001 0.001 0.001"/>
+      <mesh filename="file://$(find remy_description)/meshes/limb5_v1__1__1.stl" scale="0.001 0.001 0.001"/>
     </geometry>
     <material name="silver"/>
@@ -252,5 +252,5 @@
     <origin xyz="-0.112 -0.095 -0.0331" rpy="0 0 0"/>
     <geometry>
-      <mesh filename="file://$(find urdf2_description)/meshes/limb5_v1__2__1.stl" scale="0.001 0.001 0.001"/>
+      <mesh filename="file://$(find remy_description)/meshes/limb5_v1__2__1.stl" scale="0.001 0.001 0.001"/>
     </geometry>
     <material name="silver"/>
@@ -272,5 +272,5 @@
     <origin xyz="0.068 -0.095 -0.0331" rpy="0 0 0"/>
     <geometry>
-      <mesh filename="file://$(find urdf2_description)/meshes/limb5_v1__3__1.stl" scale="0.001 0.001 0.001"/>
+      <mesh filename="file://$(find remy_description)/meshes/limb5_v1__3__1.stl" scale="0.001 0.001 0.001"/>
     </geometry>
     <material name="silver"/>

File: remy_description/urdf/urdf2original.xacro (robot description, xacro)
@@ -1,7 +1,7 @@
 <?xml version="1.0" ?>
 <robot name="urdf2" xmlns:xacro="http://www.ros.org/wiki/xacro">
-<xacro:include filename="$(find urdf2_description)/urdf/materials.xacro" />
-<xacro:include filename="$(find urdf2_description)/urdf/urdf2.trans" />
-<xacro:include filename="$(find urdf2_description)/urdf/urdf2.gazebo" />
+<xacro:include filename="$(find remy_description)/urdf/materials.xacro" />
+<xacro:include filename="$(find remy_description)/urdf/urdf2.trans" />
+<xacro:include filename="$(find remy_description)/urdf/urdf2.gazebo" />
 <link name="base_footprint"/>
 <joint name="base_joint" type="fixed">
@@ -19,5 +19,5 @@
     <origin xyz="0 0 0" rpy="0 0 0"/>
     <geometry>
-      <mesh filename="file://$(find urdf2_description)/meshes/base_link.stl" scale="0.001 0.001 0.001"/>
+      <mesh filename="file://$(find remy_description)/meshes/base_link.stl" scale="0.001 0.001 0.001"/>
     </geometry>
     <material name="silver"/>
@@ -26,5 +26,5 @@
     <origin xyz="0 0 0" rpy="0 0 0"/>
     <geometry>
-      <mesh filename="file://$(find urdf2_description)/meshes/base_link.stl" scale="0.001 0.001 0.001"/>
+      <mesh filename="file://$(find remy_description)/meshes/base_link.stl" scale="0.001 0.001 0.001"/>
     </geometry>
   </collision>
@@ -39,5 +39,5 @@
     <origin xyz="-0.0215 0.190948 -0.125363" rpy="0 0 0"/>
     <geometry>
-      <mesh filename="file://$(find urdf2_description)/meshes/limb2_v1_1.stl" scale="0.001 0.001 0.001"/>
+      <mesh filename="file://$(find remy_description)/meshes/limb2_v1_1.stl" scale="0.001 0.001 0.001"/>
     </geometry>
     <material name="silver"/>
@@ -46,5 +46,5 @@
     <origin xyz="-0.0215 0.190948 -0.125363" rpy="0 0 0"/>
     <geometry>
-      <mesh filename="file://$(find urdf2_description)/meshes/limb2_v1_1.stl" scale="0.001 0.001 0.001"/>
+      <mesh filename="file://$(find remy_description)/meshes/limb2_v1_1.stl" scale="0.001 0.001 0.001"/>
     </geometry>
   </collision>
@@ -59,5 +59,5 @@
     <origin xyz="-0.0325 -0.0265 -1.500001" rpy="0 0 0"/>
     <geometry>
-      <mesh filename="file://$(find urdf2_description)/meshes/limb3_v1_1.stl" scale="0.001 0.001 0.001"/>
+      <mesh filename="file://$(find remy_description)/meshes/limb3_v1_1.stl" scale="0.001 0.001 0.001"/>
     </geometry>
     <material name="silver"/>
@@ -66,5 +66,5 @@
     <origin xyz="-0.0325 -0.0265 -1.500001" rpy="0 0 0"/>
     <geometry>
-      <mesh filename="file://$(find urdf2_description)/meshes/limb3_v1_1.stl" scale="0.001 0.001 0.001"/>
+      <mesh filename="file://$(find remy_description)/meshes/limb3_v1_1.stl" scale="0.001 0.001 0.001"/>
     </geometry>
   </collision>
@@ -79,5 +79,5 @@
     <origin xyz="-0.2235 -0.0 -0.074" rpy="0 0 0"/>
     <geometry>
-      <mesh filename="file://$(find urdf2_description)/meshes/limb1_v1_1.stl" scale="0.001 0.001 0.001"/>
+      <mesh filename="file://$(find remy_description)/meshes/limb1_v1_1.stl" scale="0.001 0.001 0.001"/>
     </geometry>
     <material name="silver"/>
@@ -86,5 +86,5 @@
     <origin xyz="-0.2235 -0.0 -0.074" rpy="0 0 0"/>
     <geometry>
-      <mesh filename="file://$(find urdf2_description)/meshes/limb1_v1_1.stl" scale="0.001 0.001 0.001"/>
+      <mesh filename="file://$(find remy_description)/meshes/limb1_v1_1.stl" scale="0.001 0.001 0.001"/>
     </geometry>
   </collision>
@@ -99,5 +99,5 @@
     <origin xyz="0.2245 0.0 -0.074" rpy="0 0 0"/>
     <geometry>
-      <mesh filename="file://$(find urdf2_description)/meshes/limb1_v1__1__1.stl" scale="0.001 0.001 0.001"/>
+      <mesh filename="file://$(find remy_description)/meshes/limb1_v1__1__1.stl" scale="0.001 0.001 0.001"/>
     </geometry>
     <material name="silver"/>
@@ -106,5 +106,5 @@
     <origin xyz="0.2245 0.0 -0.074" rpy="0 0 0"/>
     <geometry>
-      <mesh filename="file://$(find urdf2_description)/meshes/limb1_v1__1__1.stl" scale="0.001 0.001 0.001"/>
+      <mesh filename="file://$(find remy_description)/meshes/limb1_v1__1__1.stl" scale="0.001 0.001 0.001"/>
     </geometry>
   </collision>
@@ -119,5 +119,5 @@
     <origin xyz="0.09 0.12 -0.093" rpy="0 0 0"/>
     <geometry>
-      <mesh filename="file://$(find urdf2_description)/meshes/limb4_v1_1.stl" scale="0.001 0.001 0.001"/>
+      <mesh filename="file://$(find remy_description)/meshes/limb4_v1_1.stl" scale="0.001 0.001 0.001"/>
     </geometry>
     <material name="silver"/>
@@ -126,5 +126,5 @@
     <origin xyz="0.09 0.12 -0.093" rpy="0 0 0"/>
     <geometry>
-      <mesh filename="file://$(find urdf2_description)/meshes/limb4_v1_1.stl" scale="0.001 0.001 0.001"/>
+      <mesh filename="file://$(find remy_description)/meshes/limb4_v1_1.stl" scale="0.001 0.001 0.001"/>
     </geometry>
   </collision>
@@ -139,5 +139,5 @@
     <origin xyz="-0.09 -0.12 -0.093" rpy="0 0 0"/>
     <geometry>
-      <mesh filename="file://$(find urdf2_description)/meshes/limb4_v1__1__1.stl" scale="0.001 0.001 0.001"/>
+      <mesh filename="file://$(find remy_description)/meshes/limb4_v1__1__1.stl" scale="0.001 0.001 0.001"/>
     </geometry>
     <material name="silver"/>
@@ -146,5 +146,5 @@
     <origin xyz="-0.09 -0.12 -0.093" rpy="0 0 0"/>
     <geometry>
-      <mesh filename="file://$(find urdf2_description)/meshes/limb4_v1__1__1.stl" scale="0.001 0.001 0.001"/>
+      <mesh filename="file://$(find remy_description)/meshes/limb4_v1__1__1.stl" scale="0.001 0.001 0.001"/>
     </geometry>
   </collision>
@@ -159,5 +159,5 @@
     <origin xyz="0.09 -0.12 -0.093" rpy="0 0 0"/>
     <geometry>
-      <mesh filename="file://$(find urdf2_description)/meshes/limb4_v1__2__1.stl" scale="0.001 0.001 0.001"/>
+      <mesh filename="file://$(find remy_description)/meshes/limb4_v1__2__1.stl" scale="0.001 0.001 0.001"/>
     </geometry>
     <material name="silver"/>
@@ -166,5 +166,5 @@
     <origin xyz="0.09 -0.12 -0.093" rpy="0 0 0"/>
     <geometry>
-      <mesh filename="file://$(find urdf2_description)/meshes/limb4_v1__2__1.stl" scale="0.001 0.001 0.001"/>
+      <mesh filename="file://$(find remy_description)/meshes/limb4_v1__2__1.stl" scale="0.001 0.001 0.001"/>
     </geometry>
   </collision>
@@ -179,5 +179,5 @@
     <origin xyz="-0.09 0.12 -0.093" rpy="0 0 0"/>
     <geometry>
-      <mesh filename="file://$(find urdf2_description)/meshes/limb4_v1__3__1.stl" scale="0.001 0.001 0.001"/>
+      <mesh filename="file://$(find remy_description)/meshes/limb4_v1__3__1.stl" scale="0.001 0.001 0.001"/>
     </geometry>
     <material name="silver"/>
@@ -186,5 +186,5 @@
     <origin xyz="-0.09 0.12 -0.093" rpy="0 0 0"/>
     <geometry>
-      <mesh filename="file://$(find urdf2_description)/meshes/limb4_v1__3__1.stl" scale="0.001 0.001 0.001"/>
+      <mesh filename="file://$(find remy_description)/meshes/limb4_v1__3__1.stl" scale="0.001 0.001 0.001"/>
     </geometry>
   </collision>
@@ -199,5 +199,5 @@
     <origin xyz="0.068 0.145 -0.0331" rpy="0 0 0"/>
     <geometry>
-      <mesh filename="file://$(find urdf2_description)/meshes/limb5_v1_1.stl" scale="0.001 0.001 0.001"/>
+      <mesh filename="file://$(find remy_description)/meshes/limb5_v1_1.stl" scale="0.001 0.001 0.001"/>
     </geometry>
     <material name="silver"/>
@@ -206,5 +206,5 @@
     <origin xyz="0.068 0.145 -0.0331" rpy="0 0 0"/>
     <geometry>
-      <mesh filename="file://$(find urdf2_description)/meshes/limb5_v1_1.stl" scale="0.001 0.001 0.001"/>
+      <mesh filename="file://$(find remy_description)/meshes/limb5_v1_1.stl" scale="0.001 0.001 0.001"/>
     </geometry>
   </collision>
@@ -219,5 +219,5 @@
     <origin xyz="-0.112 0.145 -0.0331" rpy="0 0 0"/>
     <geometry>
-      <mesh filename="file://$(find urdf2_description)/meshes/limb5_v1__1__1.stl" scale="0.001 0.001 0.001"/>
+      <mesh filename="file://$(find remy_description)/meshes/limb5_v1__1__1.stl" scale="0.001 0.001 0.001"/>
     </geometry>
     <material name="silver"/>
@@ -226,5 +226,5 @@
     <origin xyz="-0.112 0.145 -0.0331" rpy="0 0 0"/>
     <geometry>
-      <mesh filename="file://$(find urdf2_description)/meshes/limb5_v1__1__1.stl" scale="0.001 0.001 0.001"/>
+      <mesh filename="file://$(find remy_description)/meshes/limb5_v1__1__1.stl" scale="0.001 0.001 0.001"/>
     </geometry>
   </collision>
@@ -239,5 +239,5 @@
     <origin xyz="-0.112 -0.095 -0.0331" rpy="0 0 0"/>
     <geometry>
-      <mesh filename="file://$(find urdf2_description)/meshes/limb5_v1__2__1.stl" scale="0.001 0.001 0.001"/>
+      <mesh filename="file://$(find remy_description)/meshes/limb5_v1__2__1.stl" scale="0.001 0.001 0.001"/>
     </geometry>
     <material name="silver"/>
@@ -246,5 +246,5 @@
     <origin xyz="-0.112 -0.095 -0.0331" rpy="0 0 0"/>
     <geometry>
-      <mesh filename="file://$(find urdf2_description)/meshes/limb5_v1__2__1.stl" scale="0.001 0.001 0.001"/>
+      <mesh filename="file://$(find remy_description)/meshes/limb5_v1__2__1.stl" scale="0.001 0.001 0.001"/>
     </geometry>
   </collision>
@@ -259,5 +259,5 @@
     <origin xyz="0.068 -0.095 -0.0331" rpy="0 0 0"/>
     <geometry>
-      <mesh filename="file://$(find urdf2_description)/meshes/limb5_v1__3__1.stl" scale="0.001 0.001 0.001"/>
+      <mesh filename="file://$(find remy_description)/meshes/limb5_v1__3__1.stl" scale="0.001 0.001 0.001"/>
     </geometry>
     <material name="silver"/>
@@ -266,5 +266,5 @@
     <origin xyz="0.068 -0.095 -0.0331" rpy="0 0 0"/>
     <geometry>
-      <mesh filename="file://$(find urdf2_description)/meshes/limb5_v1__3__1.stl" scale="0.001 0.001 0.001"/>
+      <mesh filename="file://$(find remy_description)/meshes/limb5_v1__3__1.stl" scale="0.001 0.001 0.001"/>
     </geometry>
   </collision>
